Commit message: updated stool urdfs

File: PoseEstimationDemoProject/Assets/TutorialAssets/URDFs/flisat/flisat.urdf (robot description, URDF)
Before this commit: robot flisat, 5 links, 4 joints
Links:
- link flisat_leg_1_link: geometry collision mesh filename=package://stool_description/meshes/flisat_leg.stl scale=1 1 1; visual mesh filename=package://stool_description/meshes/flisat_leg.stl scale=1 1 1
- link flisat_leg_2_link: geometry collision mesh filename=package://stool_description/meshes/flisat_leg.stl scale=1 1 1; visual mesh filename=package://stool_description/meshes/flisat_leg.stl scale=1 1 1
- link flisat_leg_3_link: geometry collision mesh filename=package://stool_description/meshes/flisat_leg.stl scale=1 1 1; visual mesh filename=package://stool_description/meshes/flisat_leg.stl scale=1 1 1
- link flisat_leg_4_link: geometry collision mesh filename=package://stool_description/meshes/flisat_leg.stl scale=1 1 1; visual mesh filename=package://stool_description/meshes/flisat_leg.stl scale=1 1 1
- link flisat_plate_link: geometry collision mesh filename=package://stool_description/meshes/flisat_plate.stl scale=1 1 1; visual mesh filename=package://stool_description/meshes/flisat_plate.stl scale=1 1 1
Joints:
- joint flisat_leg_1_joint: origin xyz=0.071207 0.071207 0.005503 rpy=-0.11938 0.11938 0 -> xyz=0.071207 0.071207 0.028303 rpy=-0.11938 0.11938 0
- joint flisat_leg_2_joint: origin xyz=0.071207 -0.071207 0.005503 rpy=0.11938 0.11938 0 -> xyz=0.071207 -0.071207 0.028303 rpy=0.11938 0.11938 0
- joint flisat_leg_3_joint: origin xyz=-0.071207 -0.071207 0.005503 rpy=0.11938 -0.11938 0 -> xyz=-0.071207 -0.071207 0.028303 rpy=0.11938 -0.11938 0
- joint flisat_leg_4_joint: origin xyz=-0.071207 0.071207 0.005503 rpy=-0.11938 -0.11938 0 -> xyz=-0.071207 0.071207 0.028303 rpy=-0.11938 -0.11938 0

File: PoseEstimationDemoProject/Assets/TutorialAssets/URDFs/flisat/stool_description/urdf/flisat.urdf (robot description, URDF)
Before this commit: robot flisat, 5 links, 4 joints
Links:
- link flisat_leg_1_link: geometry collision mesh filename=package://stool_description/meshes/flisat_leg.stl scale=1 1 1; visual mesh filename=package://stool_description/meshes/flisat_leg.stl scale=1 1 1
- link flisat_leg_2_link: geometry collision mesh filename=package://stool_description/meshes/flisat_leg.stl scale=1 1 1; visual mesh filename=package://stool_description/meshes/flisat_leg.stl scale=1 1 1
- link flisat_leg_3_link: geometry collision mesh filename=package://stool_description/meshes/flisat_leg.stl scale=1 1 1; visual mesh filename=package://stool_description/meshes/flisat_leg.stl scale=1 1 1
- link flisat_leg_4_link: geometry collision mesh filename=package://stool_description/meshes/flisat_leg.stl scale=1 1 1; visual mesh filename=package://stool_description/meshes/flisat_leg.stl scale=1 1 1
- link flisat_plate_link: geometry collision mesh filename=package://stool_description/meshes/flisat_plate.stl scale=1 1 1; visual mesh filename=package://stool_description/meshes/flisat_plate.stl scale=1 1 1
Joints:
- joint flisat_leg_1_joint: origin xyz=0.071207 0.071207 0.005503 rpy=-0.11938 0.11938 0 -> xyz=0.071207 0.071207 0.028303 rpy=-0.11938 0.11938 0
- joint flisat_leg_2_joint: origin xyz=0.071207 -0.071207 0.005503 rpy=0.11938 0.11938 0 -> xyz=0.071207 -0.071207 0.028303 rpy=0.11938 0.11938 0
- joint flisat_leg_3_joint: origin xyz=-0.071207 -0.071207 0.005503 rpy=0.11938 -0.11938 0 -> xyz=-0.071207 -0.071207 0.028303 rpy=0.11938 -0.11938 0
- joint flisat_leg_4_joint: origin xyz=-0.071207 0.071207 0.005503 rpy=-0.11938 -0.11938 0 -> xyz=-0.071207 0.071207 0.028303 rpy=-0.11938 -0.11938 0

File: PoseEstimationDemoProject/Assets/TutorialAssets/URDFs/flisat/stool_description/urdf/flisat_leg.urdf (robot description, URDF)
Before this commit: robot flisat_leg, 1 links, 0 joints
Links:
- link flisat_leg_link: geometry collision mesh filename=package://stool_description/meshes/flisat_leg.stl scale=1 1 1; visual mesh filename=package://stool_description/meshes/flisat_leg.stl scale=1 1 1

File: PoseEstimationDemoProject/Assets/TutorialAssets/URDFs/flisat_leg/flisat_leg.urdf (robot description, URDF)
Before this commit: robot flisat_leg, 1 links, 0 joints
Links:
- link flisat_leg_link: geometry collision mesh filename=package://stool_description/meshes/flisat_leg.stl scale=1 1 1; visual mesh filename=package://stool_description/meshes/flisat_leg.stl scale=1 1 1

File: PoseEstimationDemoProject/Assets/TutorialAssets/URDFs/flisat_plate/flisat_plate.urdf (robot description, URDF)
Before this commit: robot flisat_plate, 1 links, 0 joints
Links:
- link flisat_plate_link: geometry collision mesh filename=package://stool_description/meshes/flisat_plate.stl scale=1 1 1; visual mesh filename=package://stool_description/meshes/flisat_plate.stl scale=1 1 1
